Commit message: added laser scan to rviz, serial_node_struct, fixed a relative pathing issue, and added dependency on sensor_msgs

File: ROS_Workspace/src/robocar/urdf/robocar.urdf (robot description, URDF)
Before this commit: robot robocar, 9 links, 8 joints
Joints:
- joint servo_yaw: axis 0 0 1 -> 0 0 -1

Commit message: fixed urdf camera orientation, added camera calibration yaml

File: ROS_Workspace/src/robocar/urdf/robocar.urdf (robot description, URDF)
Before this commit: robot robocar, 9 links, 8 joints
Joints:
- joint camera_offset: origin xyz=0.04 0 0 -> xyz=0.04 0 0 rpy=-1.5708 0 -1.5708

Commit message: tweaked rviz, updated URDF fixed laser scan base

File: ROS_Workspace/src/robocar/urdf/robocar.urdf (robot description, URDF)
Before this commit: robot robocar, 9 links, 8 joints
Links:
- added link laser_scanner
Joints:
- added joint laser_scanner_fixed: type fixed, parent base_link, child laser_scanner, origin xyz=0.0925 0 0.121 rpy=3.141592 0 0
- joint servo_yaw: limit lower=-0.785 upper=0.785 effort=1 velocity=1 -> lower=-1.57 upper=1.57 effort=1 velocity=1
